Commit message: 미션 수정
CenterPose, HeadPose 추가, pose_pub.py 수정, mission.py 추가, goal.py 추가. 계속 수정 중

File: racecar.xacro (robot description, xacro)
@@ -26,4 +26,18 @@
     </visual>
   </link>
+  <link name="center">
+  </link>
+  <joint name="base_to_center" type="fixed">
+    <parent link="base_link"/>
+    <child link="center"/>
+    <origin xyz="${wheelbase/2} 0 0"/>
+  </joint>
+  <link name="head">
+  </link>
+  <joint name="base_to_head" type="fixed">
+    <parent link="base_link"/>
+    <child link="head"/>
+    <origin xyz="${wheelbase} 0 0"/>
+  </joint>
   <joint name="base_to_laser_model" type="fixed">
     <parent link="base_link"/>
